Commit message: Urdf y sim con sensores generales

File: install/my_agv_super/share/my_agv_super/models/myagv.urdf (robot description, URDF)
Before this commit: robot my_agv_super, 4 links, 3 joints
Links:
- removed link camera_link
- added link gps_link
- added link imu_link
- link lidar_link: mass None -> 0.114; geometry collision cylinder length=0.18 radius=0.0508; visual cylinder length=0.18 radius=0.0508
Joints:
- removed joint camera_joint
- added joint gps_joint: type fixed, parent base_link, child gps_link, origin xyz=0.10 0 0.05 rpy=0 0 0
- added joint imu_joint: type fixed, parent base_link, child imu_link, origin xyz=-0.10 0 0.05 rpy=0 0 0
- joint lidar_joint: origin xyz=${base_length/2-0.1} 0 0.05 rpy=0 0 0 -> xyz=0.066 0 0.2 rpy=0 0 0

Commit message: Fix Odom

File: install/my_agv_super/share/my_agv_super/models/myagv.urdf (robot description, URDF)
Before this commit: robot my_agv_super, 5 links, 4 joints
Links:
- link lidar_link: geometry collision cylinder length=0.08 radius=0.0508; visual cylinder length=0.18 radius=0.0508

Commit message: Slam works with bugs

File: install/my_agv_super/share/my_agv_super/models/myagv.urdf (robot description, URDF)
Before this commit: robot my_agv_super, 5 links, 4 joints
Links:
- link lidar_link: geometry collision cylinder length=0.08 radius=0.0508; visual cylinder length=0.05 radius=0.04

Commit message: Slam real ok Slam sim mov invertido

File: install/my_agv_super/share/my_agv_super/models/myagv.urdf (robot description, URDF)
Before this commit: robot my_agv_super, 5 links, 4 joints
Links:
- removed link lidar_link
- added link laser_frame, mass 0.114; collision cylinder length=0.08 radius=0.0508; visual cylinder length=0.05 radius=0.04
Joints:
- joint lidar_joint: child lidar_link -> laser_frame; origin xyz=0.066 0 0.2 rpy=0 0 0 -> xyz=0.066 0 0.05 rpy=0 0 3.14
