Commit message: backup

File: models/myagvreal.urdf (robot description, URDF)
Before this commit: robot my_agv_super, 2 links, 1 joints
Links:
- added link camera_link; visual box size=0.05 0.05 0.05
- added link imu; visual box size=0.04 0.04 0.01
- added link laser_frame; visual cylinder length=0.1 radius=0.05
- link base_up: geometry collision box size=${base_length} ${base_width} ${base_height}; visual mesh filename=package://my_agv_super/meshes/myagv_up.dae scale=1 1 1
Joints:
- added joint base_to_camera: type fixed, parent base_footprint, child camera_link, origin xyz=0.13 0 0.131 rpy=0 0 0
- added joint base_to_imu: type fixed, parent base_footprint, child imu, origin xyz=0 0 0 rpy=0 3.14159 3.14159
- added joint base_to_laser: type fixed, parent base_footprint, child laser_frame, origin xyz=0.065 0.0 0.08 rpy=0 0 3.14159

File: models/myagvros2.urdf (robot description, URDF)
Before this commit: robot my_agv_super, 5 links, 4 joints
Links:
- removed link gps_link
- removed link imu_link
- added link camera_link; visual box size=0.05 0.05 0.05
- added link imu; visual box size=0.04 0.04 0.01
- link base_link: geometry collision box size=${base_length} ${base_width} ${base_height}; visual mesh filename=package://myagv_ros2_urdf/meshes/myagv_all.dae scale=1 1 1
- link laser_frame: geometry collision cylinder length=0.05 radius=0.0508; visual cylinder length=0.05 radius=0.04
Joints:
- removed joint gps_joint
- added joint camera_joint: type fixed, parent base_footprint, child camera_link, origin xyz=0.13 0 0.131 rpy=0 0 0
- joint imu_joint: child imu_link -> imu; origin xyz=-0.10 0 0.05 rpy=0 0 0 -> xyz=0 0 0 rpy=0 3.14159 3.14159
- joint lidar_joint: origin xyz=0.066 0 0.05 rpy=0 0 3.14 -> xyz=0.065 0 0.08 rpy=0 0 3.14159

File: models/myagvsimulated.urdf (robot description, URDF)
Before this commit: robot my_agv_super, 5 links, 4 joints
Joints:
- joint lidar_joint: origin xyz=0.066 0 0.05 rpy=0 0 0 -> xyz=0.066 0 0.05 rpy=0 0 3.14
